Commit message: ares launch file and sim tests

File: ares_description/urdf/ares.urdf.xacro (robot description, xacro)
@@ -7,5 +7,5 @@
 		<color rgba="0 0 0 1"/>
 	</material>
-	<!-- <link name="base_footprint"/> -->
+	<link name="base_link"/>
 	<xacro:property name="chassisWidth" value="0.203" />
 	<xacro:property name="chassisHeight" value="0.093" />
@@ -13,5 +13,5 @@
 	<xacro:property name="wheelRadius" value="0.06" />
 	<xacro:property name="wheelWidth" value="0.05" />
-	<link name="base_link">
+	<link name="chassis">
 		<visual>
 			<geometry>
@@ -27,16 +27,18 @@
 		</collision>
 		<inertial>
-			<mass value="10"/>
-			<inertia ixx="0.11954" ixy="0.0" ixz="0.0" iyy="0.1521" iyz="0.0" izz="0.499"/>
-		</inertial>
-	</link>
-	<gazebo reference="base_link">
+			<mass value="5"/>
+			<inertia ixx="0.046204" ixy="0.0" ixz="0.0"
+               iyy="0.01717" iyz="0.0"
+               izz="0.063374" />
+		</inertial>
+	</link>
+	<gazebo reference="chassis">
     	<material>Gazebo/DarkGrey</material>
   	</gazebo>
-	<!-- <joint name="base_joint" type="fixed">
-    	<parent link="base_footprint"/>
-    	<child link="base_link"/>
+	<joint name="base_joint" type="fixed">
+    	<parent link="base_link"/>
+    	<child link="chassis"/>
     	<origin xyz="0.0 0.0 0.044250" rpy="0 0 0"/>
-  	</joint> -->
+  	</joint>
 	<link name="left_rear_wheel_link">
 		<visual>
@@ -54,9 +56,11 @@
 		<inertial>
 			<mass value="0.150"/>
-			<inertia ixx="0.000166" ixy="0.0" ixz="0.0" iyy="0.000166" iyz="0.0" izz="0.00027"/>
+			<inertia ixx="0.0002281" ixy="0.0" ixz="0.0"
+               iyy="0.0002281" iyz="0.0"
+               izz="0.00027" />
 		</inertial>
 	</link>
 	<joint name="left_rear_wheel_joint" type="continuous">
-		<parent link="base_link"/>
+		<parent link="chassis"/>
 		<child link="left_rear_wheel_link"/>
 		<axis xyz="0 0 1"/>
@@ -73,8 +77,6 @@
 	</transmission>
 	<gazebo reference="left_rear_wheel_link">
-		<mu1 value="0.1"/>
-		<mu2 value="0.1"/>
-		<kp value="500000.0"/>
-		<kd value="1.0"/>
+		<mu1 value="200.0"/>
+		<mu2 value="100.0"/>
 		<material>Gazebo/Grey</material>
 	</gazebo>
@@ -94,9 +96,11 @@
 		<inertial>
 			<mass value="0.150"/>
-			<inertia ixx="0.000166" ixy="0.0" ixz="0.0" iyy="0.000166" iyz="0.0" izz="0.00027"/>
+			<inertia ixx="0.0002281" ixy="0.0" ixz="0.0"
+               iyy="0.0002281" iyz="0.0"
+               izz="0.00027" />
 		</inertial>
 	</link>
 	<joint name="left_front_wheel_joint" type="continuous">
-		<parent link="base_link"/>
+		<parent link="chassis"/>
 		<child link="left_front_wheel_link"/>
 		<axis xyz="0 0 1"/>
@@ -112,9 +116,7 @@
 		</joint>
 	</transmission>
-	<gazebo reference="left_front_wheel_link">
-		<mu1 value="0.1"/>
-		<mu2 value="0.1"/>
-		<kp value="500000.0"/>
-		<kd value="1.0"/>
+	<gazebo reference0="left_front_wheel_link">
+		<mu1 value="0.01"/>
+		<mu2 value="0.01"/>
 		<material>Gazebo/Grey</material>
 	</gazebo>
@@ -124,22 +126,24 @@
 				<cylinder length="${wheelWidth}" radius="${wheelRadius}"/>
 			</geometry>
-			<origin rpy="0 0 0" xyz="0 0 0"/>
-			<material name="black"/>
-		</visual>
-		<collision>
-			<geometry>
-				<cylinder length="${wheelWidth}" radius="${wheelRadius}"/>
-			</geometry>
-		</collision>
-		<inertial>
-			<mass value="0.150"/>
-			<inertia ixx="0.000166" ixy="0.0" ixz="0.0" iyy="0.000166" iyz="0.0" izz="0.00027"/>
+			<origin rpy="1.57075 0 0" xyz="0 0 0"/>
+			<material name="black"/>
+		</visual>
+		<collision>
+			<geometry>
+				<cylinder length="${wheelWidth}" radius="${wheelRadius}"/>
+			</geometry>
+		</collision>
+		<inertial>
+			<mass value="0.150"/>
+			<inertia ixx="0.0002281" ixy="0.0" ixz="0.0"
+               iyy="0.0002281" iyz="0.0"
+               izz="0.00027" />
 		</inertial>
 	</link>
 	<joint name="right_rear_wheel_joint" type="continuous">
-		<parent link="base_link"/>
+		<parent link="chassis"/>
 		<child link="right_rear_wheel_link"/>
 		<axis xyz="0 0 1"/>
-		<origin rpy="1.57075 0 0" xyz="-0.089 -0.12862 0.01575"/>
+		<origin rpy="0 0 0" xyz="-0.089 -0.12862 0.01575"/>
 	</joint>
 	<transmission name="right_rear_wheel_trans">
@@ -153,8 +157,11 @@
 	</transmission>
 	<gazebo reference="right_rear_wheel_link">
-		<mu1 value="0.1"/>
-		<mu2 value="0.1"/>
-		<kp value="500000.0"/>
-		<kd value="1.0"/>
+		<mu1>0.1</mu1>
+    <mu2>0.1</mu2>
+    <kp>500000.0</kp>
+    <kd>10.0</kd>
+    <minDepth>0.001</minDepth>
+    <maxVel>0.1</maxVel>
+    <fdir1>1 0 0</fdir1>
 		<material>Gazebo/Grey</material>
 	</gazebo>
@@ -164,22 +171,25 @@
 				<cylinder length="${wheelWidth}" radius="${wheelRadius}"/>
 			</geometry>
-			<origin rpy="0 0 0" xyz="0 0 0"/>
-			<material name="black"/>
-		</visual>
-		<collision>
-			<geometry>
-				<cylinder length="${wheelWidth}" radius="${wheelRadius}"/>
-			</geometry>
-		</collision>
-		<inertial>
-			<mass value="0.150"/>
-			<inertia ixx="0.000166" ixy="0.0" ixz="0.0" iyy="0.000166" iyz="0.0" izz="0.00027"/>
+			<origin rpy="1.57075 0 0" xyz="0 0 0"/>
+			<material name="black"/>
+		</visual>
+		<collision>
+			<geometry>
+				<cylinder length="${wheelWidth}" radius="${wheelRadius}"/>
+			</geometry>
+		</collision>
+		<inertial>
+			<mass value="0.150"/>
+			<inertia ixx="0.0002281" ixy="0.0" ixz="0.0"
+               iyy="0.0002281" iyz="0.0"
+               izz="0.00027" />
 		</inertial>
 	</link>
 	<joint name="right_front_wheel_joint" type="continuous">
-		<parent link="base_link"/>
+		<parent link="chassis"/>
 		<child link="right_front_wheel_link"/>
 		<axis xyz="0 0 1"/>
-		<origin rpy="1.57075 0 0" xyz="0.089 -0.12862 0.01575"/>
+		<origin rpy="0 0 0" xyz="0.089 -0.12862 0.01575"/>
+		<dynamics friction="10"/>
 	</joint>
 	<transmission name="right_front_wheel_trans">
@@ -193,8 +203,11 @@
 	</transmission>
 	<gazebo reference="right_front_wheel_link">
-		<mu1 value="0.1"/>
-		<mu2 value="0.1"/>
-		<kp value="500000.0"/>
-		<kd value="1.0"/>
+		<mu1>10</mu1>
+    <mu2>10</mu2>
+    <kp>500000.0</kp>
+    <kd>10.0</kd>
+    <minDepth>0.001</minDepth>
+    <maxVel>0.1</maxVel>
+    <fdir1>1 0 0</fdir1>
 		<material>Gazebo/Grey</material>
 	</gazebo>
@@ -209,5 +222,5 @@
 	</link>
 	<joint name="base_to_front_handle" type="fixed">
-    	<parent link="base_link"/>
+    	<parent link="chassis"/>
     	<child link="front_handle"/>
     	<origin xyz="0.1665 0.0 0.0365" rpy="0 0 0"/>
@@ -223,8 +236,41 @@
 	</link>
 	<joint name="base_to_rear_handle" type="fixed">
-    	<parent link="base_link"/>
+    	<parent link="chassis"/>
     	<child link="rear_handle"/>
     	<origin xyz="-0.1665 0.0 0.0365" rpy="0 0 0"/>
   	</joint> -->
+	<link name="imu_link"/>
+	<joint name="imu_joint" type="fixed">
+		<parent link="chassis"/>
+		<child link="imu_link"/>
+		<origin xyz="0 0 0.006"/>
+	</joint>
+	<link name="base_scan">
+    <visual>
+      <origin xyz="0 0 0.0" rpy="0 0 0"/>
+      <geometry>
+        <mesh filename="package://ares_description/meshes/lidar.stl" scale="0.001 0.001 0.001"/>
+      </geometry>
+      <material name="black"/>
+    </visual>
+    <collision>
+      <origin xyz="0.015 0 -0.0065" rpy="0 0 0"/>
+      <geometry>
+        <cylinder length="0.0315" radius="0.055"/>
+      </geometry>
+    </collision>
+    <inertial>
+      <mass value="0.114" />
+      <origin xyz="0 0 0" />
+      <inertia ixx="0.001" ixy="0.0" ixz="0.0"
+               iyy="0.001" iyz="0.0"
+               izz="0.001" />
+    </inertial>
+  </link>
+  <joint name="scan_joint" type="fixed">
+    <parent link="chassis"/>
+    <child link="base_scan"/>
+    <origin xyz="0 0 0.093" rpy="1.57075 0 0"/>
+  </joint>
   	<gazebo>
 		<plugin name="gazebo_ros_control" filename="libgazebo_ros_control.so">

Commit message: modifying sim

File: ares_description/urdf/ares.urdf.xacro (robot description, xacro)
@@ -46,5 +46,5 @@
 				<cylinder length="${wheelWidth}" radius="${wheelRadius}"/>
 			</geometry>
-			<origin rpy="0 0 0" xyz="0 0 0"/>
+			<origin rpy="1.57075 0 0" xyz="0 0 0"/>
 			<material name="black"/>
 		</visual>
@@ -64,6 +64,6 @@
 		<parent link="chassis"/>
 		<child link="left_rear_wheel_link"/>
-		<axis xyz="0 0 1"/>
-		<origin rpy="1.57075 0 0" xyz="-0.089 0.12862 0.01575"/>
+		<axis xyz="0 1 0"/>
+		<origin rpy="0 0 0" xyz="-0.089 0.12862 0.01575"/>
 	</joint>
 	<transmission name="left_rear_wheel_trans">
@@ -77,6 +77,10 @@
 	</transmission>
 	<gazebo reference="left_rear_wheel_link">
-		<mu1 value="200.0"/>
-		<mu2 value="100.0"/>
+		<mu1 value="0.8" />
+    	<mu2 value="0.8" />
+    	<kp value="1000000.0" />
+    	<kd value="1.0" />
+    	<maxVel value="0.0" />
+  		<minDepth value="0.001"/>
 		<material>Gazebo/Grey</material>
 	</gazebo>
@@ -86,5 +90,5 @@
 				<cylinder length="${wheelWidth}" radius="${wheelRadius}"/>
 			</geometry>
-			<origin rpy="0 0 0" xyz="0 0 0"/>
+			<origin rpy="1.57075 0 0" xyz="0 0 0"/>
 			<material name="black"/>
 		</visual>
@@ -104,6 +108,6 @@
 		<parent link="chassis"/>
 		<child link="left_front_wheel_link"/>
-		<axis xyz="0 0 1"/>
-		<origin rpy="1.57075 0 0" xyz="0.089 0.12862 0.01575"/>
+		<axis xyz="0 1 0"/>
+		<origin rpy="0 0 0" xyz="0.089 0.12862 0.01575"/>
 	</joint>
 	<transmission name="left_front_wheel_trans">
@@ -116,7 +120,11 @@
 		</joint>
 	</transmission>
-	<gazebo reference0="left_front_wheel_link">
-		<mu1 value="0.01"/>
-		<mu2 value="0.01"/>
+	<gazebo reference="left_front_wheel_link">
+		<mu1 value="0.8" />
+    	<mu2 value="0.8" />
+    	<kp value="1000000.0" />
+    	<kd value="1.0" />
+    	<maxVel value="0.0" />
+  		<minDepth value="0.001"/>
 		<material>Gazebo/Grey</material>
 	</gazebo>
@@ -144,5 +152,5 @@
 		<parent link="chassis"/>
 		<child link="right_rear_wheel_link"/>
-		<axis xyz="0 0 1"/>
+		<axis xyz="0 1 0"/>
 		<origin rpy="0 0 0" xyz="-0.089 -0.12862 0.01575"/>
 	</joint>
@@ -157,11 +165,10 @@
 	</transmission>
 	<gazebo reference="right_rear_wheel_link">
-		<mu1>0.1</mu1>
-    <mu2>0.1</mu2>
-    <kp>500000.0</kp>
-    <kd>10.0</kd>
-    <minDepth>0.001</minDepth>
-    <maxVel>0.1</maxVel>
-    <fdir1>1 0 0</fdir1>
+		<mu1 value="0.8" />
+    	<mu2 value="0.8" />
+    	<kp value="1000000.0" />
+    	<kd value="1.0" />
+    	<maxVel value="0.0" />
+  		<minDepth value="0.001"/>
 		<material>Gazebo/Grey</material>
 	</gazebo>
@@ -189,7 +196,6 @@
 		<parent link="chassis"/>
 		<child link="right_front_wheel_link"/>
-		<axis xyz="0 0 1"/>
+		<axis xyz="0 1 0"/>
 		<origin rpy="0 0 0" xyz="0.089 -0.12862 0.01575"/>
-		<dynamics friction="10"/>
 	</joint>
 	<transmission name="right_front_wheel_trans">
@@ -203,11 +209,10 @@
 	</transmission>
 	<gazebo reference="right_front_wheel_link">
-		<mu1>10</mu1>
-    <mu2>10</mu2>
-    <kp>500000.0</kp>
-    <kd>10.0</kd>
-    <minDepth>0.001</minDepth>
-    <maxVel>0.1</maxVel>
-    <fdir1>1 0 0</fdir1>
+		<mu1 value="0.8" />
+    	<mu2 value="0.8" />
+    	<kp value="1000000.0" />
+    	<kd value="1.0" />
+    	<maxVel value="0.0" />
+  		<minDepth value="0.001"/>
 		<material>Gazebo/Grey</material>
 	</gazebo>
@@ -248,5 +253,5 @@
 	<link name="base_scan">
     <visual>
-      <origin xyz="0 0 0.0" rpy="0 0 0"/>
+      <origin xyz="0 0 0.0" rpy="1.57075 0 0"/>
       <geometry>
         <mesh filename="package://ares_description/meshes/lidar.stl" scale="0.001 0.001 0.001"/>
@@ -271,6 +276,66 @@
     <parent link="chassis"/>
     <child link="base_scan"/>
-    <origin xyz="0 0 0.093" rpy="1.57075 0 0"/>
+    <origin xyz="0 0 0.093" rpy="0 0 0"/>
   </joint>
+    <gazebo>
+    <plugin name="imu_plugin" filename="libgazebo_ros_imu.so">
+      <alwaysOn>true</alwaysOn>
+      <bodyName>imu_link</bodyName>
+      <frameName>imu_link</frameName>
+      <topicName>imu</topicName>
+      <serviceName>imu_service</serviceName>
+      <gaussianNoise>0.0</gaussianNoise>
+      <updateRate>0</updateRate>
+      <imu>
+        <noise>
+          <type>gaussian</type>
+          <rate>
+            <mean>0.0</mean>
+            <stddev>2e-4</stddev>
+            <bias_mean>0.0000075</bias_mean>
+            <bias_stddev>0.0000008</bias_stddev>
+          </rate>
+          <accel>
+            <mean>0.0</mean>
+            <stddev>1.7e-2</stddev>
+            <bias_mean>0.1</bias_mean>
+            <bias_stddev>0.001</bias_stddev>
+          </accel>
+        </noise>
+      </imu>
+    </plugin>
+  </gazebo>
+  <gazebo reference="base_scan">
+    <material>Gazebo/FlatBlack</material>
+    <sensor type="ray" name="lds_lfcd_sensor">
+      <pose>0 0 0 0 0 0</pose>
+      <visualize>false</visualize>
+      <update_rate>5</update_rate>
+      <ray>
+        <scan>
+          <horizontal>
+            <samples>360</samples>
+            <resolution>1</resolution>
+            <min_angle>0.0</min_angle>
+            <max_angle>6.28319</max_angle>
+          </horizontal>
+        </scan>
+        <range>
+          <min>0.120</min>
+          <max>3.5</max>
+          <resolution>0.015</resolution>
+        </range>
+        <noise>
+          <type>gaussian</type>
+          <mean>0.0</mean>
+          <stddev>0.01</stddev>
+        </noise>
+      </ray>
+      <plugin name="gazebo_ros_lds_lfcd_controller" filename="libgazebo_ros_laser.so">
+        <topicName>scan</topicName>
+        <frameName>base_scan</frameName>
+      </plugin>
+    </sensor>
+  </gazebo>
   	<gazebo>
 		<plugin name="gazebo_ros_control" filename="libgazebo_ros_control.so">

Commit message: Modification launch files, ares_remote, gmapping in simulation

File: ares_description/urdf/ares.urdf.xacro (robot description, xacro)
@@ -25,4 +25,5 @@
 				<box size="${chassisLength} ${chassisWidth} ${chassisHeight}"/>
 			</geometry>
+			<origin rpy="0 0 0" xyz="0 0 ${chassisHeight/2}"/>
 		</collision>
 		<inertial>
@@ -53,4 +54,5 @@
 				<cylinder length="${wheelWidth}" radius="${wheelRadius}"/>
 			</geometry>
+			<origin rpy="1.57075 0 0" xyz="0 0 0"/>
 		</collision>
 		<inertial>
@@ -97,4 +99,5 @@
 				<cylinder length="${wheelWidth}" radius="${wheelRadius}"/>
 			</geometry>
+			<origin rpy="1.57075 0 0" xyz="0 0 0"/>
 		</collision>
 		<inertial>
@@ -141,4 +144,5 @@
 				<cylinder length="${wheelWidth}" radius="${wheelRadius}"/>
 			</geometry>
+			<origin rpy="1.57075 0 0" xyz="0 0 0"/>
 		</collision>
 		<inertial>
@@ -185,4 +189,5 @@
 				<cylinder length="${wheelWidth}" radius="${wheelRadius}"/>
 			</geometry>
+			<origin rpy="1.57075 0 0" xyz="0 0 0"/>
 		</collision>
 		<inertial>
@@ -260,5 +265,5 @@
     </visual>
     <collision>
-      <origin xyz="0.015 0 -0.0065" rpy="0 0 0"/>
+      <origin xyz="0 0 ${0.0315/2}" rpy="0 0 0"/>
       <geometry>
         <cylinder length="0.0315" radius="0.055"/>
@@ -276,5 +281,5 @@
     <parent link="chassis"/>
     <child link="base_scan"/>
-    <origin xyz="0 0 0.093" rpy="0 0 0"/>
+    <origin xyz="0 0 0.1" rpy="0 0 0"/>
   </joint>
     <gazebo>

Commit message: Correction motor drive GroupSyncRead

File: ares_description/urdf/ares.urdf.xacro (robot description, xacro)
@@ -299,5 +299,5 @@
     <parent link="chassis"/>
     <child link="base_scan"/>
-    <origin xyz="0 0 0.1" rpy="0 0 0"/>
+    <origin xyz="0 0 0.1" rpy="0 0 1.57075"/>
   </joint>
     <gazebo>

Commit message: update description

File: ares_description/urdf/ares.urdf.xacro (robot description, xacro)
@@ -299,5 +299,5 @@
     <parent link="chassis"/>
     <child link="base_scan"/>
-    <origin xyz="0 0 0.1" rpy="0 0 1.57075"/>
+    <origin xyz="0 0 0.1" rpy="0 0 0"/>
   </joint>
     <gazebo>
