Commit message: Adding submodule explore_lite rplidar_ros, adding navigaiton, updating ares launch files, update URDF

File: ares_description/urdf/ares.urdf.xacro (robot description, xacro)
@@ -8,4 +8,5 @@
 	</material>
 	<link name="base_link"/>
+	<!--***********CHASSIS**********-->
 	<xacro:property name="chassisWidth" value="0.203" />
 	<xacro:property name="chassisHeight" value="0.093" />
@@ -16,7 +17,8 @@
 		<visual>
 			<geometry>
-				<box size="${chassisLength} ${chassisWidth} ${chassisHeight}"/>
-			</geometry>
-			<origin rpy="0 0 0" xyz="0 0 ${chassisHeight/2}"/>
+				<!-- <box size="${chassisLength} ${chassisWidth} ${chassisHeight}"/> -->
+				<mesh filename="package://ares_description/meshes/ares_body.dae" scale="0.001 0.001 0.001"/>
+			</geometry>
+			<origin rpy="0 0 1.57075" xyz="0 0 ${chassisHeight/2}"/>
 			<material name="red"/>
 		</visual>
@@ -34,7 +36,4 @@
 		</inertial>
 	</link>
-	<gazebo reference="chassis">
-    	<material>Gazebo/DarkGrey</material>
-  	</gazebo>
 	<joint name="base_joint" type="fixed">
     	<parent link="base_link"/>
@@ -42,4 +41,5 @@
     	<origin xyz="0.0 0.0 0.044250" rpy="0 0 0"/>
   	</joint>
+  	<!--***********LEFT REAR WHEEL**********-->
 	<link name="left_rear_wheel_link">
 		<visual>
@@ -69,5 +69,5 @@
 		<origin rpy="0 0 0" xyz="-0.089 0.12862 0.01575"/>
 	</joint>
-	<transmission name="left_rear_wheel_trans">
+<!-- 	<transmission name="left_rear_wheel_trans">
 		<type>transmission_interface/SimpleTransmission</type>
 		<actuator name="left_rear_wheel_motor">
@@ -77,5 +77,5 @@
 			<hardwareInterface>hardware_interface/VelocityJointInterface</hardwareInterface>
 		</joint>
-	</transmission>
+	</transmission> -->
 	<gazebo reference="left_rear_wheel_link">
 		<mu1 value="0.8" />
@@ -87,4 +87,5 @@
 		<material>Gazebo/Grey</material>
 	</gazebo>
+	<!--***********LEFT FRONT WHEEL**********-->
 	<link name="left_front_wheel_link">
 		<visual>
@@ -114,5 +115,5 @@
 		<origin rpy="0 0 0" xyz="0.089 0.12862 0.01575"/>
 	</joint>
-	<transmission name="left_front_wheel_trans">
+<!-- 	<transmission name="left_front_wheel_trans">
 		<type>transmission_interface/SimpleTransmission</type>
 		<actuator name="left_front_wheel_motor">
@@ -122,5 +123,5 @@
 			<hardwareInterface>hardware_interface/VelocityJointInterface</hardwareInterface>
 		</joint>
-	</transmission>
+	</transmission> -->
 	<gazebo reference="left_front_wheel_link">
 		<mu1 value="0.8" />
@@ -132,4 +133,5 @@
 		<material>Gazebo/Grey</material>
 	</gazebo>
+	<!--***********RIGHT REAR WHEEL**********-->
 	<link name="right_rear_wheel_link">
 		<visual>
@@ -159,5 +161,5 @@
 		<origin rpy="0 0 0" xyz="-0.089 -0.12862 0.01575"/>
 	</joint>
-	<transmission name="right_rear_wheel_trans">
+<!-- 	<transmission name="right_rear_wheel_trans">
 		<type>transmission_interface/SimpleTransmission</type>
 		<actuator name="right_rear_wheel_motor">
@@ -167,5 +169,5 @@
 			<hardwareInterface>hardware_interface/VelocityJointInterface</hardwareInterface>
 		</joint>
-	</transmission>
+	</transmission> -->
 	<gazebo reference="right_rear_wheel_link">
 		<mu1 value="0.8" />
@@ -177,4 +179,5 @@
 		<material>Gazebo/Grey</material>
 	</gazebo>
+	<!--***********RIGHT FRONT WHEEL**********-->
 	<link name="right_front_wheel_link">
 		<visual>
@@ -204,5 +207,5 @@
 		<origin rpy="0 0 0" xyz="0.089 -0.12862 0.01575"/>
 	</joint>
-	<transmission name="right_front_wheel_trans">
+<!-- 	<transmission name="right_front_wheel_trans">
 		<type>transmission_interface/SimpleTransmission</type>
 		<actuator name="right_front_wheel_motor">
@@ -212,5 +215,5 @@
 			<hardwareInterface>hardware_interface/VelocityJointInterface</hardwareInterface>
 		</joint>
-	</transmission>
+	</transmission> -->
 	<gazebo reference="right_front_wheel_link">
 		<mu1 value="0.8" />
@@ -222,50 +225,46 @@
 		<material>Gazebo/Grey</material>
 	</gazebo>
+	<!--***********GAZEBO CONTROLLER**********-->
+<!-- 	<gazebo reference="skid_steer_controller">
+  		<plugin name="skid_steer_drive_controller" filename="libgazebo_ros_skid_steer_drive.so">
+    		<updateRate>100.0</updateRate>
+    		<robotNamespace>/</robotNamespace>
+    		<odometryTopic>odom</odometryTopic>
+   			<odometryFrame>odom</odometryFrame>
+    		<leftFrontJoint>left_front_wheel_joint</leftFrontJoint>
+    		<rightFrontJoint>right_front_wheel_joint</rightFrontJoint>
+    		<leftRearJoint>left_rear_wheel_joint</leftRearJoint>
+    		<rightRearJoint>right_rear_wheel_joint</rightRearJoint>
+    		<wheelSeparation>0.25724</wheelSeparation>
+    		<wheelDiameter>0.12</wheelDiameter>
+    		<robotBaseFrame>base_link</robotBaseFrame>
+    		<torque>20000</torque>
+    		<commandTopic>cmd_vel</commandTopic>
+    		<broadcastTF>true</broadcastTF>
+  		</plugin>
+	</gazebo> -->
 	<gazebo>
-  <plugin name="skid_steer_drive_controller" filename="libgazebo_ros_skid_steer_drive.so">
-    <updateRate>100.0</updateRate>
-    <robotNamespace></robotNamespace>
-    <odometryTopic>odom</odometryTopic>
-    <odometryFrame>odom</odometryFrame>
-    <leftFrontJoint>left_front_wheel_joint</leftFrontJoint>
-    <rightFrontJoint>right_front_wheel_joint</rightFrontJoint>
-    <leftRearJoint>left_rear_wheel_joint</leftRearJoint>
-    <rightRearJoint>right_rear_wheel_joint</rightRearJoint>
-    <wheelSeparation>0.25724</wheelSeparation>
-    <wheelDiameter>0.12</wheelDiameter>
-    <robotBaseFrame>base_link</robotBaseFrame>
-    <torque>20000</torque>
-    <commandTopic>cmd_vel</commandTopic>
-    <broadcastTF>true</broadcastTF>
-  </plugin>
-</gazebo>
-<!-- 	<link name="front_handle">
-		<visual>
-			<geometry>
-				<box size="0.03 0.280 0.02"/>
-			</geometry>
-			<origin rpy="0 0 0" xyz="0.015 0 0"/>
-			<material name="black"/>
-		</visual>
-	</link>
-	<joint name="base_to_front_handle" type="fixed">
-    	<parent link="chassis"/>
-    	<child link="front_handle"/>
-    	<origin xyz="0.1665 0.0 0.0365" rpy="0 0 0"/>
-  	</joint>
-  	<link name="rear_handle">
-		<visual>
-			<geometry>
-				<box size="0.03 0.280 0.02"/>
-			</geometry>
-			<origin rpy="0 0 0" xyz="-0.015 0 0"/>
-			<material name="black"/>
-		</visual>
-	</link>
-	<joint name="base_to_rear_handle" type="fixed">
-    	<parent link="chassis"/>
-    	<child link="rear_handle"/>
-    	<origin xyz="-0.1665 0.0 0.0365" rpy="0 0 0"/>
-  	</joint> -->
+		<plugin name="turtlebot3_burger_controller" filename="libgazebo_ros_diff_drive.so">
+			<commandTopic>cmd_vel</commandTopic>
+			<odometryTopic>odom</odometryTopic>
+			<odometryFrame>odom</odometryFrame>
+			<odometrySource>world</odometrySource>
+			<publishOdomTF>true</publishOdomTF>
+			<robotBaseFrame>base_link</robotBaseFrame>
+			<publishWheelTF>false</publishWheelTF>
+			<publishTf>true</publishTf>
+			<publishWheelJointState>true</publishWheelJointState>
+			<legacyMode>false</legacyMode>
+			<updateRate>30</updateRate>
+			<leftJoint>left_front_wheel_joint</leftJoint>
+			<rightJoint>right_front_wheel_joint</rightJoint>
+			<wheelSeparation>0.25724</wheelSeparation>
+			<wheelDiameter>0.12</wheelDiameter>
+			<wheelAcceleration>1</wheelAcceleration>
+			<wheelTorque>10</wheelTorque>
+			<rosDebugLevel>na</rosDebugLevel>
+		</plugin>
+	</gazebo>
+	<!--***********IMU**********-->
 	<link name="imu_link"/>
 	<joint name="imu_joint" type="fixed">
@@ -274,91 +273,93 @@
 		<origin xyz="0 0 0.006"/>
 	</joint>
+	<gazebo reference="imu_link">
+    	<plugin name="imu_plugin" filename="libgazebo_ros_imu.so">
+      		<alwaysOn>true</alwaysOn>
+      		<bodyName>imu_link</bodyName>
+      		<frameName>imu_link</frameName>
+      		<topicName>imu</topicName>
+      		<serviceName>imu_service</serviceName>
+      		<gaussianNoise>0.0</gaussianNoise>
+      		<updateRate>5</updateRate>
+      		<imu>
+        		<noise>
+	          		<type>gaussian</type>
+	          		<rate>
+	            		<mean>0.0</mean>
+	            		<stddev>2e-4</stddev>
+	            		<bias_mean>0.0000075</bias_mean>
+	            		<bias_stddev>0.0000008</bias_stddev>
+	          		</rate>
+	          		<accel>
+	            		<mean>0.0</mean>
+	            		<stddev>1.7e-2</stddev>
+	            		<bias_mean>0.1</bias_mean>
+	            		<bias_stddev>0.001</bias_stddev>
+	          		</accel>
+        		</noise>
+      		</imu>
+    	</plugin>
+  	</gazebo>
+  	<!--***********LIDAR SCAN**********-->
 	<link name="base_scan">
-    <visual>
-      <origin xyz="0 0 0.0" rpy="1.57075 0 0"/>
-      <geometry>
-        <mesh filename="package://ares_description/meshes/lidar.stl" scale="0.001 0.001 0.001"/>
-      </geometry>
-      <material name="black"/>
-    </visual>
-    <collision>
-      <origin xyz="0 0 ${0.0315/2}" rpy="0 0 0"/>
-      <geometry>
-        <cylinder length="0.0315" radius="0.055"/>
-      </geometry>
-    </collision>
-    <inertial>
-      <mass value="0.114" />
-      <origin xyz="0 0 0" />
-      <inertia ixx="0.001" ixy="0.0" ixz="0.0"
-               iyy="0.001" iyz="0.0"
-               izz="0.001" />
-    </inertial>
-  </link>
-  <joint name="scan_joint" type="fixed">
-    <parent link="chassis"/>
-    <child link="base_scan"/>
-    <origin xyz="0 0 0.1" rpy="0 0 0"/>
-  </joint>
-    <gazebo>
-    <plugin name="imu_plugin" filename="libgazebo_ros_imu.so">
-      <alwaysOn>true</alwaysOn>
-      <bodyName>imu_link</bodyName>
-      <frameName>imu_link</frameName>
-      <topicName>imu</topicName>
-      <serviceName>imu_service</serviceName>
-      <gaussianNoise>0.0</gaussianNoise>
-      <updateRate>5</updateRate>
-      <imu>
-        <noise>
-          <type>gaussian</type>
-          <rate>
-            <mean>0.0</mean>
-            <stddev>2e-4</stddev>
-            <bias_mean>0.0000075</bias_mean>
-            <bias_stddev>0.0000008</bias_stddev>
-          </rate>
-          <accel>
-            <mean>0.0</mean>
-            <stddev>1.7e-2</stddev>
-            <bias_mean>0.1</bias_mean>
-            <bias_stddev>0.001</bias_stddev>
-          </accel>
-        </noise>
-      </imu>
-    </plugin>
-  </gazebo>
-  <gazebo reference="base_scan">
-    <material>Gazebo/FlatBlack</material>
-    <sensor type="ray" name="lds_lfcd_sensor">
-      <pose>0 0 0 0 0 0</pose>
-      <visualize>false</visualize>
-      <update_rate>5</update_rate>
-      <ray>
-        <scan>
-          <horizontal>
-            <samples>360</samples>
-            <resolution>1</resolution>
-            <min_angle>0.0</min_angle>
-            <max_angle>6.28319</max_angle>
-          </horizontal>
-        </scan>
-        <range>
-          <min>0.120</min>
-          <max>3.5</max>
-          <resolution>0.015</resolution>
-        </range>
-        <noise>
-          <type>gaussian</type>
-          <mean>0.0</mean>
-          <stddev>0.01</stddev>
-        </noise>
-      </ray>
-      <plugin name="gazebo_ros_lds_lfcd_controller" filename="libgazebo_ros_laser.so">
-        <topicName>scan</topicName>
-        <frameName>base_scan</frameName>
-      </plugin>
-    </sensor>
-  </gazebo>
+	    <visual>
+	      <origin xyz="0 0 0.0" rpy="1.57075 0 0"/>
+	      <geometry>
+	        <mesh filename="package://ares_description/meshes/lidar.stl" scale="0.001 0.001 0.001"/>
+	      </geometry>
+	      <material name="black"/>
+	    </visual>
+	    <collision>
+	      <origin xyz="0 0 ${0.0315/2}" rpy="0 0 0"/>
+	      <geometry>
+	        <cylinder length="0.0315" radius="0.055"/>
+	      </geometry>
+	    </collision>
+	    <inertial>
+	      <mass value="0.114" />
+	      <origin xyz="0 0 0" />
+	      <inertia ixx="0.001" ixy="0.0" ixz="0.0"
+	               iyy="0.001" iyz="0.0"
+	               izz="0.001" />
+	    </inertial>
+  	</link>
+  	<joint name="scan_joint" type="fixed">
+    	<parent link="chassis"/>
+    	<child link="base_scan"/>
+    	<origin xyz="0 0 0.1" rpy="0 0 0"/>
+  	</joint>
+	<gazebo reference="base_scan">
+		<material>Gazebo/FlatBlack</material>
+		<sensor type="ray" name="lds_lfcd_sensor">
+			<pose>0 0 0 0 0 0</pose>
+			<visualize>false</visualize>
+			<update_rate>5</update_rate>
+			<ray>
+				<scan>
+					<horizontal>
+						<samples>360</samples>
+						<resolution>1</resolution>
+						<min_angle>0.0</min_angle>
+						<max_angle>6.28319</max_angle>
+					</horizontal>
+				</scan>
+				<range>
+					<min>0.120</min>
+					<max>3.5</max>
+					<resolution>0.015</resolution>
+				</range>
+				<noise>
+					<type>gaussian</type>
+					<mean>0.0</mean>
+					<stddev>0.01</stddev>
+				</noise>
+			</ray>
+			<plugin name="gazebo_ros_lds_lfcd_controller" filename="libgazebo_ros_laser.so">
+				<topicName>scan</topicName>
+				<frameName>base_scan</frameName>
+			</plugin>
+		</sensor>
+	</gazebo>
+	<!--***********GAZEBO**********-->
   	<gazebo>
 		<plugin name="gazebo_ros_control" filename="libgazebo_ros_control.so">

Commit message: Some correction for exploration

File: ares_description/urdf/ares.urdf.xacro (robot description, xacro)
@@ -266,9 +266,15 @@
 		</plugin>
 	</gazebo>
-	<!--***********IMU**********-->
+	<!--***********IMU & MAGNETOMETER**********-->
 	<link name="imu_link"/>
 	<joint name="imu_joint" type="fixed">
 		<parent link="chassis"/>
 		<child link="imu_link"/>
+		<origin xyz="0 0 0.006"/>
+	</joint>
+	<link name="mag_link"/>
+	<joint name="mag_joint" type="fixed">
+		<parent link="chassis"/>
+		<child link="mag_link"/>
 		<origin xyz="0 0 0.006"/>
 	</joint>
@@ -304,5 +310,5 @@
 	<link name="base_scan">
 	    <visual>
-	      <origin xyz="0 0 0.0" rpy="1.57075 0 0"/>
+	      <origin xyz="0 0 0.0" rpy="1.57075 0 3.1415"/>
 	      <geometry>
 	        <mesh filename="package://ares_description/meshes/lidar.stl" scale="0.001 0.001 0.001"/>
@@ -327,5 +333,5 @@
     	<parent link="chassis"/>
     	<child link="base_scan"/>
-    	<origin xyz="0 0 0.1" rpy="0 0 0"/>
+    	<origin xyz="0 0 0.1" rpy="0 0 3.1415"/>
   	</joint>
 	<gazebo reference="base_scan">

Commit message: Minor change URDF

File: ares_description/urdf/ares.urdf.xacro (robot description, xacro)
@@ -310,5 +310,5 @@
 	<link name="base_scan">
 	    <visual>
-	      <origin xyz="0 0 0.0" rpy="1.57075 0 3.1415"/>
+	      <origin xyz="0 0 0.0" rpy="1.57075 0 0"/>
 	      <geometry>
 	        <mesh filename="package://ares_description/meshes/lidar.stl" scale="0.001 0.001 0.001"/>
@@ -333,5 +333,5 @@
     	<parent link="chassis"/>
     	<child link="base_scan"/>
-    	<origin xyz="0 0 0.1" rpy="0 0 3.1415"/>
+    	<origin xyz="0 0 0.1" rpy="0 0 0"/>
   	</joint>
 	<gazebo reference="base_scan">

Commit message: Fixing Bringup description

File: ares_description/urdf/ares.urdf.xacro (robot description, xacro)
@@ -310,5 +310,5 @@
 	<link name="base_scan">
 	    <visual>
-	      <origin xyz="0 0 0.0" rpy="1.57075 0 0"/>
+	      <origin xyz="0 0 0.0" rpy="1.57075 0 3.1415"/>
 	      <geometry>
 	        <mesh filename="package://ares_description/meshes/lidar.stl" scale="0.001 0.001 0.001"/>
@@ -333,5 +333,5 @@
     	<parent link="chassis"/>
     	<child link="base_scan"/>
-    	<origin xyz="0 0 0.1" rpy="0 0 0"/>
+    	<origin xyz="0 0 0.1" rpy="0 0 3.1415"/>
   	</joint>
 	<gazebo reference="base_scan">

Commit message: Preparing last tests

File: ares_description/urdf/ares.urdf.xacro (robot description, xacro)
@@ -367,4 +367,105 @@
 		</sensor>
 	</gazebo>
+	<!--***********CAMERA**********-->
+	<link name="camera">
+		<visual>
+			<geometry>
+				<box size="0.04 0.1 0.02"/>
+			</geometry>
+			<origin rpy="0 0 0" xyz="-0.02 0 0.01"/>
+			<material name="black"/>
+		</visual>
+		<collision>
+			<geometry>
+				<box size="0.04 0.1 0.04"/>
+			</geometry>
+			<origin rpy="0 0 0" xyz="0 0 0"/>
+		</collision>
+	</link>
+	<joint name="camera_joint" type="fixed">
+    	<parent link="chassis"/>
+    	<child link="camera"/>
+    	<origin xyz="0.12 0.0 0.1" rpy="-1.570 0 -1.57"/>
+  	</joint>
+<!-- 	<gazebo reference="camera">
+		<sensor type="camera" name="camera">
+			<update_rate>30.0</update_rate>
+			<camera name="head">
+				<horizontal_fov>1.3962634</horizontal_fov>
+				<image>
+					<width>800</width>
+					<height>800</height>
+					<format>R8G8B8</format>
+				</image>
+				<clip>
+					<near>0.02</near>
+					<far>300</far>
+				</clip>
+				<noise>
+					<type>gaussian</type> -->
+					<!-- Noise is sampled independently per pixel on each frame.
+					   That pixel's noise value is added to each of its color
+					   channels, which at that point lie in the range [0,1]. -->
+<!-- 					<mean>0.0</mean>
+					<stddev>0.007</stddev>
+				</noise>
+			</camera>
+			<plugin name="camera_controller" filename="libgazebo_ros_camera.so">
+				<alwaysOn>true</alwaysOn>
+				<updateRate>0.0</updateRate>
+				<cameraName>/camera</cameraName>
+				<imageTopicName>image_raw</imageTopicName>
+				<cameraInfoTopicName>camera_info</cameraInfoTopicName>
+				<frameName>camera</frameName>
+				<hackBaseline>0.07</hackBaseline>
+				<distortionK1>0.0</distortionK1>
+				<distortionK2>0.0</distortionK2>
+				<distortionK3>0.0</distortionK3>
+				<distortionT1>0.0</distortionT1>
+				<distortionT2>0.0</distortionT2>
+			</plugin>
+		</sensor>
+	</gazebo> -->
+	<gazebo reference="camera">
+  <sensor name="camera" type="depth">
+    <update_rate>20</update_rate>
+    <camera>
+      <horizontal_fov>1.047198</horizontal_fov>
+      <image>
+        <width>640</width>
+        <height>480</height>
+        <format>R8G8B8</format>
+      </image>
+      <clip>
+        <near>0.05</near>
+        <far>3</far>
+      </clip>
+    </camera>
+    <plugin name="camera_controller" filename="libgazebo_ros_openni_kinect.so">
+      <baseline>0.2</baseline>
+      <alwaysOn>true</alwaysOn>
+      <updateRate>1.0</updateRate>
+      <cameraName>camera_ir</cameraName>
+      <imageTopicName>/camera/color/image_raw</imageTopicName>
+      <cameraInfoTopicName>/camera/color/camera_info</cameraInfoTopicName>
+      <depthImageTopicName>/camera/depth/image_raw</depthImageTopicName>
+      <depthImageInfoTopicName>/camera/depth/camera_info</depthImageInfoTopicName>
+      <pointCloudTopicName>/camera/depth/points</pointCloudTopicName>
+      <frameName>camera</frameName>
+      <pointCloudCutoff>0.5</pointCloudCutoff>
+      <pointCloudCutoffMax>3.0</pointCloudCutoffMax>
+      <distortionK1>0.00000001</distortionK1>
+      <distortionK2>0.00000001</distortionK2>
+      <distortionK3>0.00000001</distortionK3>
+      <distortionT1>0.00000001</distortionT1>
+      <distortionT2>0.00000001</distortionT2>
+      <CxPrime>0</CxPrime>
+      <Cx>0</Cx>
+      <Cy>0</Cy>
+      <focalLength>0</focalLength>
+      <hackBaseline>0</hackBaseline>
+    </plugin>
+  </sensor>
+</gazebo>
 	<!--***********GAZEBO**********-->
   	<gazebo>

Commit message: minor correction

File: ares_description/urdf/ares.urdf.xacro (robot description, xacro)
@@ -368,5 +368,5 @@
 	</gazebo>
 	<!--***********CAMERA**********-->
-	<link name="camera">
+	<link name="camera_link">
 		<visual>
 			<geometry>
@@ -385,6 +385,6 @@
 	<joint name="camera_joint" type="fixed">
     	<parent link="chassis"/>
-    	<child link="camera"/>
-    	<origin xyz="0.12 0.0 0.1" rpy="-1.570 0 -1.57"/>
+    	<child link="camera_link"/>
+    	<origin xyz="0.12 0.0 0.1" rpy="0 0 0"/>
   	</joint>
 <!-- 	<gazebo reference="camera">
@@ -428,5 +428,5 @@
 	</gazebo> -->
 	<gazebo reference="camera">
-  <sensor name="camera" type="depth">
+  <sensor name="camera_link" type="depth">
     <update_rate>20</update_rate>
     <camera>
